Commit message: things are looking ok

File: STEP3_inference/assets/xarm_arm/xarm6_robot.urdf (robot description, URDF)
Before this commit: robot xarm6, 8 links, 7 joints
Links:
- removed link world
- added link link_eef, mass 0.0
- added link xarm_grasptarget_vis, mass 0.0
- link link1: geometry collision mesh filename=package://xarm_description/meshes/xarm6/collision/link1_vha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; visual mesh filename=package://xarm_description/meshes/xarm6/visual/link1.obj
- link link2: geometry collision mesh filename=package://xarm_description/meshes/xarm6/collision/link2_vha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; visual mesh filename=package://xarm_description/meshes/xarm6/visual/link2.obj
- link link3: geometry collision mesh filename=package://xarm_description/meshes/xarm6/collision/link3_vha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; visual mesh filename=package://xarm_description/meshes/xarm6/visual/link3.obj
- link link4: geometry collision mesh filename=package://xarm_description/meshes/xarm6/collision/link4_vha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; visual mesh filename=package://xarm_description/meshes/xarm6/visual/link4.obj
- link link5: geometry collision mesh filename=package://xarm_description/meshes/xarm6/collision/link5_vha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; visual mesh filename=package://xarm_description/meshes/xarm6/visual/link5.obj
- link link6: geometry collision mesh filename=package://xarm_description/meshes/xarm6/collision/link6_vha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; visual mesh filename=package://xarm_description/meshes/xarm6/visual/link6.obj
- link link_base: geometry collision mesh filename=package://xarm_description/meshes/xarm6/collision/base_vhac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; visual mesh filename=package://xarm_description/meshes/xarm6/visual/base.obj
Joints:
- removed joint world_joint
- added joint joint_eef: type fixed, parent link6, child link_eef, origin xyz=0 0 0 rpy=0 0 0
- added joint xarm_grasptarget_hand: type fixed, parent link_eef, child xarm_grasptarget_vis, origin xyz=0 -0.08 0.105 rpy=0 0 0
